File: sjc_hub.kicad_pcb (KiCad board)
At the start: 2 copper layers, 65 x 100 mm, 39 parts, among them J1 PWR_IN+, J10 RS-485 B, J11 SENS A, J2 PWR_IN-, J3 SENS B, J5 SENSORS OUT, J6 P_{GND}, J7 V_{DC}, J8 RS-485 IN, J9 RS-485 A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

Commit message: pcb updates
Other:
- board text added: "Network Hub"
- board text added: "SJC"
- board text removed: "CraneControl"
- board text removed: "SJC Connections"
